Commit message: LiDAR を MID-360 化し全天球カメラ認識（物体分類・信号認識）を追加
- Gazebo MID-360: ROS2 ネイティブの LCAS livox plugin (ODE MultiRayShape) に置き換え。
  自作の格子最近傍方式で出ていた上向き自己遮蔽・幾何歪みを解消。VLP-16 版は退避。
- Webots: MID-360 近似(tiltAngle で仰角中心 +22.5°)。トピック/フレームを汎用名
  (/lidar/points, lidar_link)に統一。
- 信号認識を全天球カメラ前提に: 全周 N 分割の透視ビューで検出、方向で重複統合、
  バッチ推論、LiDAR と組み合わせ 3D 位置推定(traffic_light_localizer)。
- LiDAR 検出物体の画像分類 object_classifier を追加(全天球クロップ→YOLOv8、late fusion)。
  トラック ID キャッシュ+レート上限で間引き。YOLO 失敗は FATAL(classic 自動フォールバック禁止)。
- 画像認識を simulation / webots_simulation に image_recognition 引数で統合(既定 ON、波及)。
  webots_city を ROS2 認識対応に(city_robot.wbt: 車+歩行者+信号)。
- pointcloud_to_autoware: 混在データ型クラッシュ修正(read_points_numpy→read_points)。
- scan pattern CSV(~40MB)は .gitignore で除外。取得手順を docs に記載。
- 各種ドキュメント更新。

Co-Authored-By: Claude Opus 4.8 (1M context) <noreply@anthropic.com>

File: urdf/turtlebot3_waffle_3d.urdf.xacro (robot description, xacro)
@@ -1,9 +1,9 @@
 <?xml version="1.0" ?>
 <!--
-  TurtleBot3 Waffle + 3D LiDAR (Velodyne VLP-16 style) description, used by
-  robot_state_publisher to provide TF (including base_link -> velodyne_link).
+  TurtleBot3 Waffle + 3D LiDAR description, used by
+  robot_state_publisher to provide TF (including base_link -> lidar_link).
   The Gazebo sensor itself lives in the SDF model
   (susumu_object_perception/models/turtlebot3_waffle_3d/model.sdf); this file only adds the
-  matching velodyne_link frame so TF and the SDF agree.
+  matching lidar_link frame so TF and the SDF agree.
 -->
 <robot name="turtlebot3_waffle_3d" xmlns:xacro="http://ros.org/wiki/xacro">
@@ -11,14 +11,14 @@
   <xacro:include filename="$(find turtlebot3_description)/urdf/turtlebot3_waffle.urdf"/>
   <!-- 3D LiDAR frame, mounted on top of base_link (matches model.sdf pose) -->
-  <joint name="velodyne_joint" type="fixed">
+  <joint name="lidar_joint" type="fixed">
     <origin xyz="0 0 0.20" rpy="0 0 0"/>
     <parent link="base_link"/>
-    <child link="velodyne_link"/>
+    <child link="lidar_link"/>
   </joint>
-  <link name="velodyne_link">
+  <link name="lidar_link">
     <visual>
       <origin xyz="0 0 0" rpy="0 0 0"/>
       <geometry>
-        <cylinder radius="0.0516" length="0.0717"/>
+        <box size="0.065 0.065 0.060"/>
       </geometry>
       <material name="black"/>
@@ -27,12 +27,12 @@
       <origin xyz="0 0 0" rpy="0 0 0"/>
       <geometry>
-        <cylinder radius="0.0516" length="0.0717"/>
+        <box size="0.065 0.065 0.060"/>
       </geometry>
     </collision>
     <inertial>
-      <mass value="0.83"/>
+      <mass value="0.265"/>
       <origin xyz="0 0 0"/>
-      <inertia ixx="0.001" ixy="0.0" ixz="0.0"
-               iyy="0.001" iyz="0.0" izz="0.001"/>
+      <inertia ixx="0.0002" ixy="0.0" ixz="0.0"
+               iyy="0.0002" iyz="0.0" izz="0.0002"/>
     </inertial>
   </link>
